File: IR_PCB_hw/IR_PCB.kicad_pcb (KiCad board)
At the start: 2 copper layers, 65.5 x 60.5 mm, 111 parts, among them Q1 NSS20101, Q10 SI2303, Q11 SI2303, Q12 SI2303, Q13 SI2303, Q2 NSS20101, Q3 M28S, Q4 M28S, Q5 TSOP48xx, Q6 TSOP48xx, Q7 SI2303, Q8 TSOP48xx, Q9 SI2303

Commit message: Silks done
Parts:
- moved R3 3.10 mm to (161.6, 93.7), turned to -90 degrees
- moved R2 2.90 mm to (161.6, 96.7), turned to 90 degrees
- moved R19 1.60 mm to (148.3, 96.8)
- moved R20 1.60 mm to (149.9, 96.8), turned to -90 degrees
- moved Q9 0.61 mm to (145.5, 100.4)
- moved XL10 0.50 mm to (143.3, 104.0)
- moved C11 0.30 mm to (157.5, 79.9)
- moved Q12 0.30 mm to (158.1, 95.6)
- moved C12 0.30 mm to (159.1, 79.9)
- moved R21 0.30 mm to (155.4, 95.6)
- turned R6 to 0 degrees
- turned R7 to 0 degrees
Routing:
- net GND: track 0.00 -> 176.6 mm, vias 0 -> 67
- net +3v3: track 0.00 -> 157.7 mm, vias 0 -> 4
- net +PwrMCU: track 0.00 -> 67.6 mm, vias 0 -> 4
- net /IR_RCVR: track 0.00 -> 50.9 mm, vias 0 -> 1
- net Net-(D12-PadA): track 0.00 -> 30.9 mm
- net /LED_PWM4: track 0.00 -> 30.4 mm
- net /LED_PWM2: track 0.00 -> 30.1 mm
- net Net-(D11-PadA): track 0.00 -> 28.4 mm
- net /LED_PWM1: track 0.00 -> 25.6 mm
- net /LED_PWM3: track 0.00 -> 25.0 mm
- net /IR_LED_DAC: track 0.00 -> 23.9 mm, vias 0 -> 1
- net /LED_FRONT2: track 0.00 -> 23.2 mm, vias 0 -> 1
- net Net-(D10-PadA): track 0.00 -> 23.2 mm
- net /LED_PWM4_IN: track 0.00 -> 22.7 mm, vias 0 -> 1
- net /IR_TX_OUT: track 0.00 -> 21.9 mm
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- added copper zone on B.Cu, net GND
- added copper zone on F.Cu, net GND
Other:
- board text added: "+"
- board text added: "+3v3"
- board text added: "-"
- board text added: "GND"
- board text added: "IR LED"
- board text added: "IRRX"
- board text added: "IRTX"
- board text added: "In1"
- board text added: "In2"
- board text added: "In3"
- board text added: "LED1"
- board text added: "LED2"
- board text added: "LED3"
- board text added: "LED4"
- board text added: "LEDF1"
- board text added: "LEDF2"
- board text added: "Out1"
- board text added: "Out2"
- board text added: "Out3"
- board text added: "PWR"
- board text added: "RX"
- board text added: "TX"

Commit message: Sent to factory
Other:
- board text added: "IR PCB v1"
Changed lines of the file:
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@@
     (allow_soldermask_bridges_in_footprints yes)
     (pcbplotparams
-      (layerselection 0x00010fc_ffffffff)
+      (layerselection 0x00010f0_ffffffff)
       (plot_on_all_layers_selection 0x0000000_00000000)
       (disableapertmacros false)
-      (usegerberextensions false)
+      (usegerberextensions true)
       (usegerberattributes true)
       (usegerberadvancedattributes true)
-      (creategerberjobfile true)
+      (creategerberjobfile false)
       (dashed_line_dash_ratio 12.000000)
       (dashed_line_gap_ratio 3.000000)
@@
       (plotinvisibletext false)
       (sketchpadsonfab false)
-      (subtractmaskfromsilk false)
+      (subtractmaskfromsilk true)
       (outputformat 1)
       (mirror false)
-      (drillshape 1)
+      (drillshape 0)
       (scaleselection 1)
-      (outputdirectory "")
+      (outputdirectory "Factory")
     )
   )
@@
     (effects (font (size 1 0.6) (thickness 0.15) bold) (justify left bottom mirror))
   )
+  (gr_text "IR PCB v1" (at 156.95 86.3) (layer "B.SilkS")
+    (effects (font (size 2 1) (thickness 0.25) bold italic) (justify left bottom mirror))
+  )
   (gr_text "GND" (at 127.95 81.65 90) (layer "B.SilkS")
