File: IR_PCB_hw/IR_PCB.kicad_pcb (KiCad board)
At the start: 2 copper layers, 65.5 x 60.5 mm, 111 parts, among them Q1 NSS20101, Q10 SI2303, Q11 SI2303, Q12 SI2303, Q13 SI2303, Q2 NSS20101, Q3 M28S, Q4 M28S, Q5 TSOP48xx, Q6 TSOP48xx, Q7 SI2303, Q8 TSOP48xx, Q9 SI2303

Commit message: Layout started
Parts:
- removed Q12, Q13: SI2303, SOT:SOT23-3
- added C22: 0.1u, Capacitors:CAP_0402_Fab, F.Cu at (220.9, 116.5)
- added C23: 10u, Capacitors:CAP_0603_Silks, F.Cu at (206.6, 145.4)
- added C24: 0.1u, Capacitors:CAP_0402_Fab, F.Cu at (220.9, 118.9)
- added C25: 10u, Capacitors:CAP_0805, F.Cu at (190.3, 147.0)
- added C26: 10u, Capacitors:CAP_0603_Silks, F.Cu at (206.6, 148.1)
- added DA2: LM1117GS-3.3, SOT:SOT223, F.Cu at (226.8, 113.5)
- added DD2: W25Q32JV, SO_DIL_TSSOP:SO8_208MIL, F.Cu at (207.7, 133.5)
- added DD3: MAX98357A, QFN_DFN:QFN-16_EP_3x3_Pitch0.5mm, F.Cu at (244.6, 125.1)
- added HOLE13: HOLE_METALLED, PCB:Hole4_out5d3mm, F.Cu at (155.2, 93.8)
- added HOLE14: HOLE_METALLED, PCB:Hole4_out5d3mm, F.Cu at (155.2, 124.2)
- added HOLE15: HOLE_METALLED, PCB:Hole4_out5d3mm, F.Cu at (124.8, 124.2)
- added HOLE16: HOLE_METALLED, PCB:Hole4_out5d3mm, F.Cu at (124.8, 93.8)
- added R25: 10k, Resistors:RES_0402_Fab, F.Cu at (195.5, 127.4)
- added R26: 100R, Resistors:RES_0402_Fab, F.Cu at (195.5, 129.8)
- added R27: 100R, Resistors:RES_0402_Fab, F.Cu at (195.5, 132.1)
- added TP1: TESTPOINT, PCB:TESTPOINT_1MM, F.Cu at (244.0, 144.0)
- added TP2: TESTPOINT, PCB:TESTPOINT_1MM, F.Cu at (244.0, 146.0)
- added TP3: TESTPOINT, PCB:TESTPOINT_1MM, F.Cu at (246.0, 142.0)
- added TP4: TESTPOINT, PCB:TESTPOINT_1MM, F.Cu at (246.0, 144.0)
- added TP5: TESTPOINT, PCB:TESTPOINT_1MM, F.Cu at (246.0, 146.0)
- added XL21: SOCKET_3, Connectors:PLS-3, F.Cu at (176.8, 132.3)
- added XL22: SOCKET_3, Connectors:PLS-3, F.Cu at (176.8, 136.0)
- added XL23: SOCKET_3, Connectors:PLS-3, F.Cu at (176.8, 139.7)
- added XL24: SOCKET_3, Connectors:PLS-3, F.Cu at (176.8, 143.4)
- C10: value 0.1u -> 10u
- C11, C14, C16, C2, C20, C4, C7, C9: footprint Capacitors:CAP_0603_Silks -> Capacitors:CAP_0402_Fab
- C12: value 1u -> 0.1u; footprint Capacitors:CAP_0603_Silks -> Capacitors:CAP_0402_Fab
- C13: value 47u -> 0.1u; footprint Capacitors:CAP_1206 -> Capacitors:CAP_0402_Fab
- C15: value 0.1u -> 18pF; footprint Capacitors:CAP_0603_Silks -> Capacitors:CAP_0402_Fab
- C17: value 10u -> 47u; footprint Capacitors:CAP_0805 -> Capacitors:CAP_1206
- C18, C5: value 10u -> 0.1u; footprint Capacitors:CAP_0603_Silks -> Capacitors:CAP_0402_Fab
- C3: value 18pF -> 2u2
- C6, C8: value 0.1u -> 1u; footprint Capacitors:CAP_0603_Silks -> Capacitors:CAP_0402_Fab
- D1: value L-C191LBCT -> TSAL6200; footprint LEDs:LED_0603 -> LEDs:LED5mmR
- D2: value TSAL6200 -> L-C191LBCT; footprint LEDs:LED5mmR -> LEDs:LED_0603
- DA1: value LM1117GS-3.3 -> 74VHC1GT125; footprint SOT:SOT223 -> SOT:SOT23-5
- DD1: value STM32F072RxTx -> GD32E103CB; footprint LQFP_TQFP:LQFP64 -> LQFP_TQFP:LQFP48
- HOLE1, HOLE10, HOLE11, HOLE12, HOLE2, HOLE3, HOLE4, HOLE5, HOLE6, HOLE7, HOLE8, HOLE9: footprint PCB:Oval7d7x5d7wHole5d5x3d5 -> PCB:Hole2d7_out4d2mm
- Q1, Q2: value NSS20101 -> M28S; footprint SOT:SC89-3 -> SOT:SOT23-3
- Q10, Q11, Q7, RP3, RP4: moved to F.Cu
- Q3, Q4: value M28S -> TSOP48xx; footprint SOT:SOT23-3 -> Sensors:TSOP48xx; moved to F.Cu
- Q5, Q8: value TSOP48xx -> SI2303; footprint Sensors:TSOP48xx -> SOT:SOT23-3
- R1: value 1k -> 10k; footprint Resistors:RES_0603 -> Resistors:RES_0402_Fab
- R10, R6: value 100R -> 1k; footprint Resistors:RES_0603 -> Resistors:RES_0402_Fab; moved to F.Cu
- R11, R16: value 10k -> 51R; footprint Resistors:RES_0603 -> Resistors:RES_0402_Fab; moved to F.Cu
- R12: value 100R -> 51R; footprint Resistors:RES_0603 -> Resistors:RES_0402_Fab; moved to F.Cu
- R13, R8, R9: value 51R -> 100R; footprint Resistors:RES_0603 -> Resistors:RES_0402_Fab
- R14, R19, R24: value 100R -> 10k; footprint Resistors:RES_0603 -> Resistors:RES_0402_Fab; moved to F.Cu
- R15, R22: value 10k -> 100R; footprint Resistors:RES_0603 -> Resistors:RES_0402_Fab; moved to F.Cu
- R17, R18, R20, R21, R23, R4: footprint Resistors:RES_0603 -> Resistors:RES_0402_Fab; moved to F.Cu
- R2: value 10k -> 5k1; footprint Resistors:RES_0603 -> Resistors:RES_0402_Fab; moved to F.Cu
- R3: value DNM -> 5k1; footprint Resistors:RES_0603 -> Resistors:RES_0402_Fab; moved to F.Cu
- R5: footprint Resistors:RES_0603 -> Resistors:RES_0402_Fab
- R7: value 100R -> 2R0; footprint Resistors:RES_0603 -> Resistors:RES_0402_Fab; moved to F.Cu
- XL1: value SOCKET_2 -> SOCKET_6; footprint Connectors:PLS-2 -> Connectors:PLS-6_LOCK
- XL10: footprint Connectors:SLD_2_2D5 -> Connectors:PLS-2
- XL11: value SOCKET_3 -> SOCKET_2; footprint Connectors:PLS-3 -> Connectors:PLS-2
- XL12, XL13: value SOCKET_3 -> SOCKET_1; footprint Connectors:PLS-3 -> Connectors:PLS-1Oval
- XL20: value SOCKET_3 -> SOCKET_2; footprint Connectors:PLS-3 -> Connectors:SLD_2_2D5
- XL3: value SOCKET_4 -> SOCKET_2; footprint Connectors:PLS-4 -> Connectors:PLS-2
- XL4: value SOCKET_6 -> USB_C; footprint Connectors:PLS-6_LOCK -> Connectors:USBC_24PF-009
- XL5: footprint Connectors:PLS-4 -> Connectors:PLS-4-NoHole; moved to F.Cu
- XL6: value SOCKET_2 -> SOCKET_4; footprint Connectors:PLS-2 -> Connectors:PLS-4-NoHole
- XL9: value SOCKET_2 -> SOCKET_3; footprint Connectors:PLS-2 -> Connectors:PLS-3-PAD
- moved RP3 142.1 mm to (242.0, 146.0), turned to 0 degrees
- moved C19 136.9 mm to (244.5, 135.6), turned to 0 degrees
- moved RP1 131.3 mm to (242.0, 142.0)
- moved C21 124.6 mm to (244.5, 139.2), turned to 0 degrees
- moved XL13 114.4 mm to (240.2, 124.6), turned to 0 degrees
- moved Q8 110.9 mm to (228.9, 124.4), turned to 0 degrees
- moved Q5 108.9 mm to (224.8, 124.4), turned to 0 degrees
- moved RP2 107.9 mm to (242.0, 144.0)
- moved C17 106.9 mm to (244.5, 132.1), turned to 0 degrees
- moved C20 101.2 mm to (220.9, 114.2), turned to 0 degrees
- moved XL5 99.8 mm to (233.1, 110.2), turned to 0 degrees
- moved XL12 97.4 mm to (236.9, 124.6), turned to 0 degrees
- moved Q10 97.0 mm to (233.1, 124.4)
- moved Q7 94.9 mm to (224.8, 128.3)
- moved Q11 93.4 mm to (233.1, 128.3)
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Connections:
- C13 pad 1: Net-(Q6-Vs) -> +PwrMCU
- C14 pad 1: Net-(Q6-Vs) -> +PwrMCU
- C15 pad 1: Net-(Q5-Vs) -> Net-(C15-Pad1)
- C16 pad 1: +BATT -> Net-(Q3-Vs)
- C17 pad 1: +BATT -> Net-(Q3-Vs)
- C18 pad 1: +3v3 -> Net-(Q4-Vs)
- C19 pad 1: Net-(Q5-Vs) -> Net-(Q4-Vs)
- C20 pad 1: Net-(Q8-Vs) -> Net-(Q6-Vs)
- C21 pad 1: Net-(Q8-Vs) -> Net-(Q6-Vs)
- C3 pad 1: Net-(DD1-OSCIN/PF0) -> Net-(C3-Pad1)
- C4 pad 1: Net-(C4-Pad1) -> Net-(DD1-OSCIN)
- C5 pad 1: +PwrMCU -> /+NPX_PWR
- D1 pad A: Net-(D1-PadA) -> +3v3
- D1 pad C: GND -> /IR_TX_OUT
- D2 pad A: +3v3 -> Net-(D2-PadA)
- D2 pad C: /IR_TX_OUT -> GND
- DA1 pad 2: +3v3 -> /NPX_CTRL
- DA1 pad 3: +BATT -> GND
- DD1 pad 10: unconnected-(DD1-ADC12/MISO2/PC2-Pad10) -> /NPX_CTRL
- DD1 pad 11: unconnected-(DD1-ADC13/MOSI2/PC3-Pad11) -> /IR_RCVR
- DD1 pad 12: GND -> /UART_TX
- DD1 pad 13: +PwrMCU -> /UART_RX
- DD1 pad 14: Net-(DD1-ADC0/TX4/T2C1ETR/WKUP1/PA0) -> /IR_LED_DAC
- DD1 pad 15: /LED_FRONT1 -> /Output1
- DD1 pad 16: /LED_FRONT2 -> /LED_PWM1_IN
- DD1 pad 17: /IR_RCVR -> /LED_PWM2_IN
- DD1 pad 18: GND -> /LED_PWM3_IN
- DD1 pad 19: +PwrMCU -> /LED_PWM4_IN
- DD1 pad 2: unconnected-(DD1-WKUP2/RTC_OUT/PC13-Pad2) -> /AU_SDMODE
- DD1 pad 20: /IR_LED_DAC -> /Input1
- DD1 pad 21: unconnected-(DD1-ADC5/T2C1ETR/DAC2/SCK1/PA5-Pad21) -> /Input2
- DD1 pad 22: unconnected-(DD1-ADC6/T16C1/T3C1/MISO1/PA6-Pad22) -> /Input3
- DD1 pad 23: unconnected-(DD1-ADC7/T14C1/T17C1/T1C1N/T3C2/MOSI1/PA7-Pad23) -> GND
- DD1 pad 24: unconnected-(DD1-ADC14/TX3/PC4-Pad24) -> +PwrMCU
- DD1 pad 25: unconnected-(DD1-ADC15/WKUP5/RX3/PC5-Pad25) -> /AU_LRCK
- DD1 pad 26: unconnected-(DD1-PB0/T3C3/T1C2N/CK3/ADC8-Pad26) -> /AU_BCLK
- DD1 pad 27: unconnected-(DD1-PB1/T3C4/T14C1/T1C3N/ADC9-Pad27) -> /Buzzer
- DD1 pad 28: unconnected-(DD1-PB2-Pad28) -> /AU_SDIN
- DD1 pad 29: unconnected-(DD1-PB10/SCK2/SCL2/TX3/T2C3-Pad29) -> /Output2
- DD1 pad 3: unconnected-(DD1-OC32IN/PC14-Pad3) -> /Output3
- DD1 pad 30: unconnected-(DD1-PB11/SDA2/RX3/T2C4-Pad30) -> Net-(DD1-PA9)
- DD1 pad 31: GND -> Net-(DD1-PA10)
- DD1 pad 32: +PwrMCU -> /USB_D-
- DD1 pad 33: unconnected-(DD1-PB12/CK3-Pad33) -> /USB_D+
- DD1 pad 34: /Output1 -> /SWDIO
- DD1 pad 35: /Output2 -> GND
- DD1 pad 36: /Output3 -> +PwrMCU
- DD1 pad 37: /LED_PWM1_IN -> /SWCLK
- DD1 pad 38: /LED_PWM2_IN -> /FLASH_NSS
- DD1 pad 39: /LED_PWM3_IN -> /FLASH_SCK
- DD1 pad 40: /LED_PWM4_IN -> /FLASH_MISO
- DD1 pad 41: /Buzzer -> /FLASH_MOSI
- DD1 pad 42: /UART_TX -> /FLASH_IO2
- DD1 pad 43: /UART_RX -> /FLASH_IO3
- DD1 pad 44: unconnected-(DD1-T1C4/USBDM/PA11-Pad44) -> GND
- DD1 pad 45: unconnected-(DD1-T1ETR/USBDP/PA12-Pad45) -> /LED_FRONT1
- DD1 pad 46: /SWDIO -> /LED_FRONT2
- DD1 pad 5: Net-(DD1-OSCIN/PF0) -> Net-(DD1-OSCIN)
- DD1 pad 6: Net-(DD1-OSCOUT/PF1) -> Net-(DD1-OSCOUT)
- DD1 pad 8: unconnected-(DD1-ADC10/PC0-Pad8) -> GND
- DD1 pad 9: unconnected-(DD1-ADC11/PC1-Pad9) -> +PwrMCU
- Q10 pad 1: /LED_PWM2_IN -> GND
- Q10 pad 2: +3v3 -> +BATT
- Q10 pad 3: /LED_PWM2 -> /+PWR_IN
- Q11 pad 1: /LED_PWM3_IN -> /LED_PWM4_IN
- Q11 pad 3: /LED_PWM3 -> /LED_PWM4
- Q3 pad 1: /IR_LED_IN -> /IR_RCVR
- Q3 pad 2: /IR_INTERM -> GND
- Q3 pad 3: /IR_TX_OUT -> Net-(Q3-Vs)
- Q4 pad 1: /IR_INTERM -> /IR_RCVR
- Q4 pad 3: /IR_TX_OUT -> Net-(Q4-Vs)
- Q5 pad 1: /IR_RCVR -> /LED_PWM1_IN
- Q5 pad 2: GND -> +3v3
- Q5 pad 3: Net-(Q5-Vs) -> /LED_PWM1
- Q7 pad 1: /LED_PWM1_IN -> /LED_PWM2_IN
- Q7 pad 3: /LED_PWM1 -> /LED_PWM2
- Q8 pad 1: /IR_RCVR -> /LED_PWM3_IN
- Q8 pad 2: GND -> +3v3
- Q8 pad 3: Net-(Q8-Vs) -> /LED_PWM3
- Q9 pad 1: GND -> /Buzzer
- Q9 pad 2: +BATT -> +3v3
- Q9 pad 3: /+PWR_IN -> /BuzzerOut
- R1 pad 1: Net-(D1-PadA) -> /IR_LED_DAC
- R1 pad 2: Net-(DD1-ADC0/TX4/T2C1ETR/WKUP1/PA0) -> /IR_LED_IN
- R10 pad 1: /LED_PWM1 -> Net-(C15-Pad1)
- R10 pad 2: Net-(D5-PadA) -> Net-(DD1-OSCOUT)
- R11 pad 1: +3v3 -> Net-(Q3-Vs)
- R11 pad 2: /LED_PWM1_IN -> +3v3
- R12 pad 1: /LED_PWM2 -> Net-(Q4-Vs)
- R12 pad 2: Net-(D6-PadA) -> +3v3
- R13 pad 1: Net-(Q8-Vs) -> /LED_PWM1
- R13 pad 2: +3v3 -> Net-(D5-PadA)
- R14 pad 1: /LED_PWM3 -> +3v3
- R14 pad 2: Net-(D7-PadA) -> /LED_PWM1_IN
- R15 pad 1: /IR_RCVR -> /LED_PWM2
- R15 pad 2: +3v3 -> Net-(D6-PadA)
- R16 pad 1: +3v3 -> Net-(Q6-Vs)
- R16 pad 2: /LED_PWM2_IN -> +3v3
- R17 pad 1: /LED_PWM4 -> /LED_PWM3
- R17 pad 2: Net-(D8-PadA) -> Net-(D7-PadA)
- R18 pad 1: +3v3 -> /IR_RCVR
- R18 pad 2: /LED_PWM3_IN -> +3v3
- R19 pad 1: /LED_PWM1 -> +3v3
- R19 pad 2: Net-(D9-PadA) -> /LED_PWM2_IN
- R2 pad 1: /IR_LED_DAC -> GND
- R2 pad 2: /IR_LED_IN -> /USB_CC1
- R20 pad 1: /LED_PWM2 -> /LED_PWM4
- R20 pad 2: Net-(D10-PadA) -> Net-(D8-PadA)
- R21 pad 2: /Buzzer -> /LED_PWM3_IN
- R22 pad 1: +3v3 -> /LED_PWM1
- R22 pad 2: /LED_PWM4_IN -> Net-(D9-PadA)
- R23 pad 1: /LED_PWM3 -> /LED_PWM2
- R23 pad 2: Net-(D11-PadA) -> Net-(D10-PadA)
- R24 pad 1: /LED_PWM4 -> +3v3
- R24 pad 2: Net-(D12-PadA) -> /Buzzer
- R3 pad 1: /IR_LED_TIM -> /USB_CC2
- R3 pad 2: /IR_LED_IN -> GND
- R5 pad 1: Net-(C4-Pad1) -> +5vUSB
- R5 pad 2: Net-(DD1-OSCOUT/PF1) -> Net-(DD1-PA9)
- R6 pad 1: /LED_FRONT1 -> Net-(D2-PadA)
- R6 pad 2: Net-(D3-PadA) -> Net-(DD1-PA10)
- R7 pad 1: /LED_FRONT2 -> +5vUSB
- R7 pad 2: Net-(D4-PadA) -> Net-(C3-Pad1)
- R8 pad 1: Net-(Q5-Vs) -> /LED_FRONT1
- R8 pad 2: +3v3 -> Net-(D3-PadA)
- R9 pad 1: Net-(Q6-Vs) -> /LED_FRONT2
- R9 pad 2: +3v3 -> Net-(D4-PadA)
- XL1 pad 2: /IR_TX_OUT -> /SWCLK
- XL10 pad 1: GND -> Net-(D4-PadA)
- XL10 pad 2: /+PWR_IN -> GND
- XL11 pad 1: GND -> Net-(D4-PadA)
- XL11 pad 2: Net-(D6-PadA) -> GND
- XL12 pad 1: GND -> /SPK_P
- XL13 pad 1: GND -> /SPK_M
- XL14 pad 2: +3v3 -> Net-(D6-PadA)
- XL14 pad 3: /IR_RCVR -> Net-(D5-PadA)
- XL15 pad 2: Net-(D8-PadA) -> Net-(D6-PadA)
- XL15 pad 3: Net-(D7-PadA) -> Net-(D5-PadA)
- XL16 pad 2: Net-(D8-PadA) -> +3v3
- XL16 pad 3: Net-(D7-PadA) -> /IR_RCVR
- XL17 pad 2: Net-(D10-PadA) -> +3v3
- XL17 pad 3: Net-(D9-PadA) -> /IR_RCVR
- XL18 pad 2: Net-(D10-PadA) -> Net-(D8-PadA)
- XL18 pad 3: Net-(D9-PadA) -> Net-(D7-PadA)
- XL19 pad 2: Net-(D12-PadA) -> Net-(D8-PadA)
- XL19 pad 3: Net-(D11-PadA) -> Net-(D7-PadA)
- XL20 pad 2: Net-(D12-PadA) -> /+PWR_IN
- XL3 pad 1: GND -> +3v3
- XL3 pad 2: /Input1 -> /IR_TX_OUT
- XL5 pad 2: /Output1 -> /Input1
- XL5 pad 3: /Output2 -> /Input2
- XL5 pad 4: /Output3 -> /Input3
- XL6 pad 1: Net-(D3-PadA) -> GND
- XL6 pad 2: GND -> /Output1
- XL8 pad 1: Net-(D4-PadA) -> Net-(D3-PadA)
- XL9 pad 1: Net-(D4-PadA) -> GND
- XL9 pad 2: GND -> /NPX_DATA
- XTAL1 pad 1: Net-(DD1-OSCIN/PF0) -> Net-(DD1-OSCIN)
- XTAL1 pad 2: Net-(C4-Pad1) -> Net-(C15-Pad1)
Routing:
- net GND: track 176.6 -> 0.00 mm, vias 67 -> 0
- net +3v3: track 157.7 -> 0.00 mm, vias 4 -> 0
- net +PwrMCU: track 67.6 -> 0.00 mm, vias 4 -> 0
- net /IR_RCVR: track 50.9 -> 0.00 mm, vias 1 -> 0
- net Net-(D12-PadA): track 30.9 -> 0.00 mm
- net /LED_PWM4: track 30.4 -> 0.00 mm
- net /LED_PWM2: track 30.1 -> 0.00 mm
- net Net-(D11-PadA): track 28.4 -> 0.00 mm
- net /LED_PWM1: track 25.6 -> 0.00 mm
- net /LED_PWM3: track 25.0 -> 0.00 mm
- net /IR_LED_DAC: track 23.9 -> 0.00 mm, vias 1 -> 0
- net /LED_FRONT2: track 23.2 -> 0.00 mm, vias 1 -> 0
- net Net-(D10-PadA): track 23.2 -> 0.00 mm
- net /LED_PWM4_IN: track 22.7 -> 0.00 mm, vias 1 -> 0
- net /IR_TX_OUT: track 21.9 -> 0.00 mm
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- removed copper zone on B.Cu, net GND
- removed copper zone on F.Cu, net GND
Other:
- board size 65.5 x 60.5 mm -> 49.2 x 49 mm

Commit message: Layout in progress
Parts:
- removed C11: 0.1u, Capacitors:CAP_0402_Fab
- removed TP1: TESTPOINT, PCB:TESTPOINT_1MM
- removed XL11: SOCKET_2, Connectors:PLS-2
- removed XL12, XL13: SOCKET_1, Connectors:PLS-1Oval
- removed XL6: SOCKET_4, Connectors:PLS-4-NoHole
- added D13: PMEG2020, Diodes:SOD323, F.Cu at (129.4, 109.6)
- added R29: 10k, Resistors:RES_0402_Fab, F.Cu at (130.4, 111.0)
- C6, C7, DA1, DA2, DD2, DD3, Q10, Q9, R1, R24, R4, RP2, RP3: moved to B.Cu
- XL1: footprint Connectors:PLS-6_LOCK -> Connectors:PLS-6-NoHole
- XL10: footprint Connectors:PLS-2 -> Connectors:SLD_2_2D5_SMD
- XL14, XL16, XL18, XL21, XL23: footprint Connectors:PLS-3 -> Connectors:SLD_3_2D5_SMD; moved to B.Cu
- XL2: footprint Connectors:PLS-2 -> Connectors:SLD_2_2D5_SMD; moved to B.Cu
- XL5: value SOCKET_4 -> SOCKET_5; footprint Connectors:PLS-4-NoHole -> Connectors:SLD_5_2D5_SMD
- XL7: value SOCKET_2 -> SOCKET_3; footprint Connectors:PLS-2 -> Connectors:SLD_3_2D5_SMD; moved to B.Cu
- XL8: value SOCKET_2 -> SOCKET_3; footprint Connectors:PLS-2 -> Connectors:PLS-3
- XL9: footprint Connectors:PLS-3-PAD -> Connectors:SLD_3_2D5_SMD
- moved C21 130.3 mm to (120.2, 100.2)
- moved C17 129.4 mm to (116.2, 115.4)
- moved RP4 127.2 mm to (118.8, 119.6)
- moved DD3 126.4 mm to (118.2, 125.4), turned to 180 degrees
- moved RP3 126.0 mm to (118.8, 119.6), turned to 180 degrees
- moved C19 122.9 mm to (123.4, 114.8), turned to -90 degrees
- moved D2 113.2 mm to (131.4, 114.6), turned to -90 degrees
- moved RP2 107.5 mm to (151.4, 86.2), turned to 180 degrees
- moved RP1 106.4 mm to (151.4, 86.2)
- moved C16 105.1 mm to (115.8, 110.2), turned to 90 degrees
- moved C20 104.5 mm to (116.6, 107.2), turned to -30 degrees
- moved Q10 102.8 mm to (131.2, 111.0), turned to 180 degrees
- moved C18 102.2 mm to (118.7, 109.6), turned to -150 degrees
- moved XL5 99.2 mm to (134.0, 115.2), turned to 90 degrees
- moved XL20 92.3 mm to (128.8, 114.0), turned to 90 degrees
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Connections:
- net /Input1 renamed /Gpio1
- net /Input2 renamed /Gpio2
- net /Input3 renamed /Gpio3
- C22 pad 1: /+AU_PWR -> +PwrUnst
- C23 pad 2: /+AU_PWR -> +PwrUnst
- C24 pad 1: +BATT -> +PwrUnst
- C25 pad 1: +BATT -> +PwrUnst
- C5 pad 1: /+NPX_PWR -> +PwrUnst
- DA1 pad 5: /+NPX_PWR -> +PwrUnst
- DA2 pad 3: +BATT -> +PwrUnst
- DD1 pad 15: /Output1 -> unconnected-(DD1-PA5-Pad15)
- DD1 pad 29: /Output2 -> /Gpio4
- DD1 pad 3: /Output3 -> unconnected-(DD1-PC14-Pad3)
- DD3 pad 7: /+AU_PWR -> +PwrUnst
- DD3 pad 8: /+AU_PWR -> +PwrUnst
- Q10 pad 1: GND -> +5vUSB
- Q10 pad 2: +BATT -> +PwrUnst
- XL10 pad 1: Net-(D4-PadA) -> /SPK_P
- XL10 pad 2: GND -> /SPK_M
- XL14 pad 2: Net-(D6-PadA) -> /LED_PWM2
- XL14 pad 3: Net-(D5-PadA) -> /LED_PWM1
- XL15 pad 2: Net-(D6-PadA) -> /LED_PWM2
- XL15 pad 3: Net-(D5-PadA) -> /LED_PWM1
- XL18 pad 2: Net-(D8-PadA) -> /LED_PWM4
- XL18 pad 3: Net-(D7-PadA) -> /LED_PWM3
- XL19 pad 2: Net-(D8-PadA) -> /LED_PWM4
- XL19 pad 3: Net-(D7-PadA) -> /LED_PWM3
- XL21 pad 2: Net-(D10-PadA) -> /LED_PWM2
- XL21 pad 3: Net-(D9-PadA) -> /LED_PWM1
- XL22 pad 2: Net-(D10-PadA) -> /LED_PWM2
- XL22 pad 3: Net-(D9-PadA) -> /LED_PWM1
- XL23 pad 2: Net-(D12-PadA) -> /LED_PWM4
- XL23 pad 3: Net-(D11-PadA) -> /LED_PWM3
- XL24 pad 2: Net-(D12-PadA) -> /LED_PWM4
- XL24 pad 3: Net-(D11-PadA) -> /LED_PWM3
- XL7 pad 1: Net-(D3-PadA) -> GND
- XL7 pad 2: GND -> /LED_FRONT1
- XL8 pad 1: Net-(D3-PadA) -> GND
- XL8 pad 2: GND -> /LED_FRONT1
- XL9 pad 3: /+NPX_PWR -> +PwrUnst
Other:
- board size 49.2 x 49 mm -> 49.5 x 49 mm

Commit message: PCBv3 sent to factory
Parts:
- added Logo1: Logo, Pictures:KiberiadaTYUKF, B.Cu at (120.8, 115.5)
- C10: footprint Capacitors:CAP_0603_Silks -> Capacitors:CAP_0603_Fab
- C22, C24, C5, Q11, Q5, R14, R25, R3, R5, R6, TP2, TP3, TP4, TP5: moved to B.Cu
- C23, C26: footprint Capacitors:CAP_0603_Silks -> Capacitors:CAP_0603_Fab; moved to B.Cu
- C25: footprint Capacitors:CAP_0805 -> Capacitors:CAP_0603_Fab; moved to B.Cu
- C3: footprint Capacitors:CAP_0603_Silks -> Capacitors:CAP_0402_Fab
- L1: footprint Inductors:IND_0402 -> Inductors:IND_0402_Fab; moved to B.Cu
- moved C23 53.8 mm to (131.7, 113.4), turned to -90 degrees
- moved C3 53.0 mm to (131.5, 112.3), turned to 180 degrees
- moved R14 47.9 mm to (137.5, 103.3)
- moved R7 47.4 mm to (131.5, 111.0)
- moved Q5 46.9 mm to (137.7, 101.0)
- moved R2 45.9 mm to (133.3, 99.2)
- moved R25 43.3 mm to (135.0, 108.4), turned to 180 degrees
- moved R3 43.3 mm to (133.8, 106.4)
- moved R5 43.0 mm to (137.5, 104.8)
- moved R6 42.6 mm to (138.4, 106.6), turned to 90 degrees
- moved C22 41.9 mm to (131.9, 116.1), turned to -90 degrees
- moved C5 41.4 mm to (133.4, 101.9)
- moved Q11 40.1 mm to (133.8, 111.0), turned to 180 degrees
- moved TP5 39.5 mm to (133.1, 118.2), turned to 180 degrees
- moved C25 38.2 mm to (136.3, 111.8), turned to -90 degrees
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Connections:
- XL1 pad 1: +3v3 -> +PwrMCU
Routing:
- net GND: track 0.00 -> 281.0 mm, vias 0 -> 19
- net +3v3: track 0.00 -> 112.8 mm, vias 0 -> 13
- net /LED_PWM2: track 0.00 -> 56.0 mm, vias 0 -> 2
- net +PwrMCU: track 0.00 -> 54.4 mm, vias 0 -> 4
- net /LED_PWM4: track 0.00 -> 49.0 mm, vias 0 -> 4
- net /LED_PWM1: track 0.00 -> 48.1 mm, vias 0 -> 2
- net /IR_RCVR: track 0.00 -> 47.7 mm, vias 0 -> 2
- net /LED_PWM3: track 0.00 -> 44.8 mm, vias 0 -> 3
- net +PwrUnst: track 0.00 -> 35.8 mm, vias 0 -> 4
- net /LED_FRONT1: track 0.00 -> 30.3 mm, vias 0 -> 2
- net /AU_SDMODE: track 0.00 -> 22.2 mm, vias 0 -> 3
- net /Gpio1: track 0.00 -> 22.1 mm, vias 0 -> 2
- net /SPK_P: track 0.00 -> 21.9 mm, vias 0 -> 2
- net +5vUSB: track 0.00 -> 20.9 mm, vias 0 -> 3
- net /Gpio2: track 0.00 -> 20.2 mm, vias 0 -> 2
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- added copper zone on B.Cu, net +3v3
- added copper zone on F.Cu, net +3v3
- added copper zone on In2.Cu, net +3v3
- added copper zone on B.Cu, net +PwrUnst
- added copper zone on F.Cu, net +PwrUnst
- added copper zone on B.Cu, net GND
- added copper zone on F.Cu, net GND
- added copper zone on In1.Cu, net GND
- added copper zone on In2.Cu, net GND
Other:
- copper layers 2 -> 4
- board text added: "+5V"
- board text added: "GPIO1"
- board text added: "GPIO2"
- board text added: "Кибериада ТЮКФ"
- board text added: "Произведено в России"
- board text added: "Турнир юных киберфизиков"
- board text removed: "IR PCB v1"
- board text removed: "In1"
- board text removed: "In2"
- board text removed: "In3"
- board text removed: "Out1"
- board text removed: "Out2"
- board text removed: "Out3"
- board text removed: "PWR"
- board text removed: "RX"
- board text removed: "TX"

Commit message: PCB v 3.1
Parts:
- moved DD2 0.30 mm to (142.3, 104.4)
- moved L1 0.30 mm to (147.5, 102.0)
- moved Q5 0.30 mm to (138.0, 101.0)
- moved C6 0.30 mm to (145.7, 103.0)
- moved C7 0.30 mm to (145.7, 100.9)
- moved R1 0.30 mm to (145.7, 108.9)
- moved R4 0.30 mm to (145.7, 105.8)
- moved TP5 0.22 mm to (133.3, 118.1)
- moved Q1 0.20 mm to (148.0, 109.1)
- moved Q2 0.20 mm to (148.0, 105.8)
Routing:
- net /USB_D-: track 8.72 -> 11.7 mm, vias 2 -> 3
- net /USB_D+: track 10.5 -> 12.4 mm, vias 2 -> 4
- net +PwrMCU: track 54.4 -> 56.3 mm
- net +3v3: track 112.8 -> 111.5 mm
- net /Gpio4: track 12.0 -> 13.0 mm
- net /LED_PWM4_IN: track 19.5 -> 18.6 mm
- net Net-(DD1-PA10): track 2.19 -> 2.94 mm
- net GND: track 281.0 -> 281.7 mm
- net /AU_LRCK: track 18.9 -> 19.4 mm
