File: IR_PCB_hw/IR_PCB.kicad_sch (KiCad schematic)
At the start: 74 parts, among them Q1 NSS20101, Q2 NSS20101, Q3 M28S, Q4 M28S, Q5 TSOP48xx, Q6 TSOP48xx, Q7 TSOP48xx, Q8 IRLML6401

Commit message: Layout done
Parts:
- removed C11, C9: 0.1u, Capacitors:CAP_0603_Silks, symbol Tittar_kl:C
- removed Q7: TSOP48xx, Sensors:TSOP48xx, symbol Sensors:TSOP48xx
- removed R5: 51R, Resistors:RES_0603, symbol Tittar_kl:R
- added BZ1: PS-9627, Installation:BUZZER_HC0903, symbol Tittar_kl:BUZZER
- added C13, C19, C21: 47u, Capacitors:CAP_1206, symbol Tittar_kl:C
- added C15, C16, C2, C20: 0.1u, Capacitors:CAP_0603_Silks, symbol Tittar_kl:C
- added C17: 10u, Capacitors:CAP_0805, symbol Tittar_kl:C
- added C18: 10u, Capacitors:CAP_0603_Silks, symbol Tittar_kl:C
- added DA1: LM1117GS-3.3, SOT:SOT223, symbol Power_kl:LD1117
- added HOLE1, HOLE10, HOLE11, HOLE12, HOLE2, HOLE3, HOLE4, HOLE5, HOLE6, HOLE7, HOLE8, HOLE9: HOLE_METALLED, PCB:Oval7d7x5d7wHole5d5x3d5, symbol pcb_details:HOLE_METALLED
- added L1: BLM15AG102, Inductors:IND_0402, symbol Tittar_kl:L
- added Q10, Q11, Q12, Q13, Q7: SI2303, SOT:SOT23-3, symbol Transistors_kl:P_3PIN
- added Q8: TSOP48xx, Sensors:TSOP48xx, symbol Sensors:TSOP48xx
- added R11, R16, R18, R21, R22: 10k, Resistors:RES_0603, symbol Tittar_kl:R
- added R13: 51R, Resistors:RES_0603, symbol Tittar_kl:R
- added RP1, RP2, RP3, RP4: REFPOINT, PCB:REF_POINT_1MM, symbol pcb_details:REFPOINT
- added XL5: SOCKET_4, Connectors:PLS-4, symbol Connectors_kl:SOCKET_4
- C1: renamed from C12; value 220uF -> 470uF; footprint Capacitors:CAP_05xxR_horiz -> Capacitors:CAP_D; PN EWK1CM221E11OT -> TAJD477K006RNJ; Price (none) -> 45; URL https://www.chipdip.ru/product0/9001022319 -> (none)
- Q9: renamed from Q8; value IRLML6401 -> SI2303; Price 5 -> 4; URL (none) -> https://www.chipdip.ru/product/si2301a
- XL3: renamed from XL19; footprint (none) -> Connectors:PLS-4
- renumbered C6 to C10, C7 to C11, C8 to C12, C10 to C14, C13 to C3, C14 to C4, C1 to C5, C2 to C6, C3 to C7, C4 to C8, C5 to C9, Q4 to Q3, Q3 to Q4, R11 to R10, R13 to R14, R6 to R15, R14 to R17, R15 to R19, R3 to R2, R16 to R20, R17 to R23, R18 to R24, R4 to R3, R2 to R4, R19 to R5, R9 to R6, R10 to R7, R7 to R9, XL2 to XL1, XL18 to XL10, XL10 to XL11, XL4 to XL13, XL5 to XL14, XL11 to XL15, XL13 to XL16, XL14 to XL17, XL15 to XL18, XL16 to XL19, XL3 to XL2, XL17 to XL20, XL1 to XL4
Connections:
- net +3v3: now also R15.2, XL4.1, C18.1, C2.1, DA1.2 (OUT), DA1.PAD (OUT), L1.2, Q10.2 (S), Q11.2 (S), Q12.2 (S), Q13.2 (S), Q7.2 (S), R11.1, R13.2, R16.1, R18.1, R21.1, R22.1; no longer R15.1
- net +BATT: now also C16.1, C17.1, DA1.3 (IN)
- net +PwrMCU: now also L1.1; no longer XL4.1
- net GND: now also XL6.2, XL7.2, XL8.2, XL9.2, BZ1.1, C13.2, C15.2, C16.2, C17.2, C18.2, C19.2, C2.2, C20.2, C21.2, DA1.1 (GND), HOLE1.H, HOLE10.H, HOLE11.H, HOLE12.H, HOLE2.H, HOLE3.H, HOLE4.H, HOLE5.H, HOLE6.H, HOLE7.H, HOLE8.H, HOLE9.H, Q8.2 (GND), XL5.1; no longer XL6.1, XL7.1, XL8.1, XL9.1
- net IR_RCVR: now also R15.1, Q8.1 (OUT); no longer R15.2
- net LED_PWM1: now also R19.1, Q7.3 (D); no longer DD1.37 (T3C1/PC6)
- net LED_PWM2: now also R20.1, Q10.3 (D); no longer DD1.38 (T3C2/PC7)
- net LED_PWM3: now also R23.1, Q11.3 (D); no longer DD1.39 (T3C3/PC8)
- net LED_PWM4: now also R24.1, Q13.3 (D); no longer DD1.40 (T3C4/PC9)
- net UART_RX: now also DD1.43 (T1C3/RX1/PA10); no longer DD1.59 (PB7/SDA1/T17C1N/RX1)
- net UART_TX: now also DD1.42 (T1C2/TX1/PA9); no longer DD1.58 (PB6/SCL1/T16C1N/TX1)
- net at D3.A, R6.2: now also XL6.1, XL7.1; no longer XL6.2, XL7.2
- net at C14.1, Q6.3 (Vs), R9.1: now also C13.1
- net at D4.A, R7.2: now also XL8.1, XL9.1; no longer XL8.2, XL9.2
- net at R8.1: now also Q5.3 (Vs), C15.1, C19.1
- net at R1.2: now also DD1.14 (ADC0/TX4/T2C1ETR/WKUP1/PA0)
- net LED_FRONT2: now reaches DD1.16 (ADC2/T15C1/T2C3/TX2/PA2)
- net LED_FRONT2: now also R7.1
- net Output1: now reaches DD1.34 (PB13/SCK2/SCL2/T1C1N)
- net Output1: now also XL5.2
- net Output2: now reaches DD1.35 (PB14/MISO2/SDA2/T1C2N/T15C1)
- net Output2: now also XL5.3
- net Output3: now reaches DD1.36 (PB15/MOSI2/T1C3N/T15C1N/T15C2)
- net Output3: now also XL5.4
- net LED_PWM10 renamed LED_FRONT1
- net LED_FRONT1: now also R6.1; no longer R7.1
- net LED_PWM5 renamed Buzzer
- net Buzzer: now also Q12.1 (G), R21.2; no longer R19.1
- removed net LED_PWM6: DD1.42 (T1C2/TX1/PA9), R20.1
- removed net LED_PWM7: DD1.43 (T1C3/RX1/PA10), R23.1
- net LED_PWM8: no longer names the net of DD1.44 (T1C4/USBDM/PA11)
- net LED_PWM8: no longer R24.1
- removed net LED_PWM9: DD1.14 (ADC0/TX4/T2C1ETR/WKUP1/PA0), R6.1
- new net: C20.1, C21.1, Q8.3 (Vs), R13.1
- new net BuzzerOut: BZ1.2, Q12.3 (D)
- new net LED_PWM1_IN: DD1.37 (T3C1/PC6), Q7.1 (G), R11.2
- new net LED_PWM2_IN: DD1.38 (T3C2/PC7), Q10.1 (G), R16.2
- new net LED_PWM3_IN: DD1.39 (T3C3/PC8), Q11.1 (G), R18.2
- new net LED_PWM4_IN: DD1.40 (T3C4/PC9), Q13.1 (G), R22.2
- no-connect marks 8 -> 29
Other:
- note added: "Inputs 5V Tolerant"
- note added: "MCU"
- note added: "Outputs Open-Drain 5V Tolerant"
- note added: "Periphery TIM1 Ch1 - Buzzer TIM2 Ch1 - SysLED Ch2 - LED_Front1 Ch3 - LED_Front2 TIM3 - Indication LEDs TIM6, TIM7 - IR TX TIM14 - System Timer TIM15 - IR RX TIM16, TIM17 - spare IR TX"
- note added: "Power"
- note added: "Power Input: [5; 16]v"
- note added: "Sound"
- note added: "System LED"
- note removed: "Inputs (5V Tolerant)"
- note removed: "Power Input"
- title: (none) -> IR PCB
- moved on the sheet: C1, C10, C11, C12, C14, C3, C4, C5, C6, C7, C8, C9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

Commit message: + BOM
Parts:
- BZ1: Price 10 -> 25
- C13, C19, C21: Price 0.5 -> 25
- C17: Price 0.5 -> 2
- Q1, Q2: Price (none) -> 40
- Q3, Q4, R3, RP1, RP2, RP3, RP4, XL1, XL10, XL11, XL12, XL13, XL14, XL15, XL16, XL17, XL18, XL19, XL2, XL20, XL3, XL5, XL6, XL7, XL8, XL9: now left out of the parts list
- Q5, Q6, Q8: Price (none) -> 120
- XL4: Price (none) -> 4
Changed lines of the file:
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@@
   )
   (symbol (lib_id "Connectors_kl:SOCKET_3") (at 219.71 180.34 0) (mirror y) (unit 1)
-    (in_bom yes) (on_board yes) (dnp no)
+    (in_bom no) (on_board yes) (dnp no)
     (property "Reference" "XL12" (at 220.98 185.42 0)
       (effects (font (size 1.016 1.016)) (justify left))
@@
       (effects (font (size 1.524 1.524)) hide)
     )
-    (property "Price" "0.5" (at 383.54 148.59 0)
+    (property "Price" "25" (at 383.54 148.59 0)
       (effects (font (size 1.524 1.524)) hide)
     )
@@
       (effects (font (size 1.524 1.524)) hide)
     )
-    (property "Price" "0.5" (at 335.28 163.83 0)
+    (property "Price" "25" (at 335.28 163.83 0)
       (effects (font (size 1.524 1.524)) hide)
     )
@@
       (effects (font (size 1.524 1.524)) hide)
     )
+    (property "Price" "120" (at 364.49 166.37 0)
+      (effects (font (size 1.27 1.27)) hide)
+    )
     (pin "1")
     (pin "2")
@@
   )
   (symbol (lib_id "pcb_details:REFPOINT") (at 302.26 210.82 0) (unit 1)
-    (in_bom yes) (on_board yes) (dnp no)
+    (in_bom no) (on_board yes) (dnp no)
     (property "Reference" "RP1" (at 306.07 209.55 0)
       (effects (font (size 1.524 1.524)) (justify left))
@@
       (effects (font (size 1.524 1.524)) hide)
     )
+    (property "Price" "4" (at 20.32 40.64 0)
+      (effects (font (size 1.27 1.27)) hide)
+    )
     (pin "1")
     (pin "2")
@@
   )
   (symbol (lib_id "Connectors_kl:SOCKET_3") (at 207.01 245.11 0) (unit 1)
-    (in_bom yes) (on_board yes) (dnp no)
+    (in_bom no) (on_board yes) (dnp no)
     (property "Reference" "XL17" (at 205.74 250.19 0)
       (effects (font (size 1.016 1.016)) (justify left))
@@
   )
   (symbol (lib_id "Connectors_kl:SOCKET_2") (at 43.18 166.37 0) (mirror y) (unit 1)
-    (in_bom yes) (on_board yes) (dnp no)
+    (in_bom no) (on_board yes) (dnp no)
     (property "Reference" "XL10" (at 44.45 171.45 0)
       (effects (font (size 1.016 1.016)) (justify left))
@@
       (effects (font (size 1.524 1.524)) hide)
     )
+    (property "Price" "120" (at 316.23 153.67 0)
+      (effects (font (size 1.27 1.27)) hide)
+    )
     (pin "1")
     (pin "2")
@@
       (effects (font (size 1.524 1.524)) hide)
     )
-    (property "Price" "10" (at 387.35 237.49 0)
+    (property "Price" "25" (at 387.35 237.49 0)
       (effects (font (size 1.524 1.524)) hide)
     )
@@
       (effects (font (size 1.524 1.524)) hide)
     )
-    (property "Price" "0.5" (at 383.54 176.53 0)
+    (property "Price" "25" (at 383.54 176.53 0)
       (effects (font (size 1.524 1.524)) hide)
     )
@@
   )
   (symbol (lib_id "Transistors_kl:NPN") (at 298.45 109.22 0) (unit 1)
-    (in_bom yes) (on_board yes) (dnp no) (fields_autoplaced)
+    (in_bom no) (on_board yes) (dnp no) (fields_autoplaced)
     (property "Reference" "Q4" (at 302.26 108.585 0)
       (effects (font (size 1.27 1.27)) (justify left))
@@
   )
   (symbol (lib_id "Connectors_kl:SOCKET_3") (at 219.71 245.11 0) (mirror y) (unit 1)
-    (in_bom yes) (on_board yes) (dnp no)
+    (in_bom no) (on_board yes) (dnp no)
     (property "Reference" "XL18" (at 220.98 250.19 0)
       (effects (font (size 1.016 1.016)) (justify left))
@@
   )
   (symbol (lib_id "Connectors_kl:SOCKET_3") (at 207.01 273.05 0) (unit 1)
-    (in_bom yes) (on_board yes) (dnp no)
+    (in_bom no) (on_board yes) (dnp no)
     (property "Reference" "XL19" (at 205.74 278.13 0)
       (effects (font (size 1.016 1.016)) (justify left))
@@
   )
   (symbol (lib_id "Connectors_kl:SOCKET_3") (at 219.71 208.28 0) (mirror y) (unit 1)
-    (in_bom yes) (on_board yes) (dnp no)
+    (in_bom no) (on_board yes) (dnp no)
     (property "Reference" "XL16" (at 220.98 213.36 0)
       (effects (font (size 1.016 1.016)) (justify left))
@@
   )
   (symbol (lib_id "Connectors_kl:SOCKET_2") (at 354.33 109.22 0) (unit 1)
-    (in_bom yes) (on_board yes) (dnp no)
+    (in_bom no) (on_board yes) (dnp no)
     (property "Reference" "XL8" (at 354.33 113.03 0)
       (effects (font (size 1.016 1.016)) (justify left))
@@
       (effects (font (size 1.524 1.524)) hide)
     )
-    (property "Price" "0.5" (at 46.99 205.74 0)
+    (property "Price" "2" (at 46.99 205.74 0)
       (effects (font (size 1.524 1.524)) hide)
     )
@@
   )
   (symbol (lib_id "pcb_details:REFPOINT") (at 302.26 223.52 0) (unit 1)
-    (in_bom yes) (on_board yes) (dnp no)
+    (in_bom no) (on_board yes) (dnp no)
     (property "Reference" "RP2" (at 306.07 222.25 0)
       (effects (font (size 1.524 1.524)) (justify left))
@@
   )
   (symbol (lib_name "REFPOINT_1") (lib_id "pcb_details:REFPOINT") (at 302.26 217.17 0) (unit 1)
-    (in_bom yes) (on_board yes) (dnp no)
+    (in_bom no) (on_board yes) (dnp no)
     (property "Reference" "RP3" (at 306.07 215.9 0)
       (effects (font (size 1.524 1.524)) (justify left))
@@
   )
   (symbol (lib_id "Connectors_kl:SOCKET_2") (at 372.11 109.22 0) (mirror y) (unit 1)
-    (in_bom yes) (on_board yes) (dnp no)
+    (in_bom no) (on_board yes) (dnp no)
     (property "Reference" "XL9" (at 372.11 113.03 0)
       (effects (font (size 1.016 1.016)) (justify left))
@@
       (effects (font (size 1.524 1.524)) hide)
     )
+    (property "Price" "120" (at 364.49 138.43 0)
+      (effects (font (size 1.27 1.27)) hide)
+    )
     (pin "1")
     (pin "2")
@@
   )
   (symbol (lib_id "Connectors_kl:SOCKET_3") (at 207.01 180.34 0) (unit 1)
-    (in_bom yes) (on_board yes) (dnp no)
+    (in_bom no) (on_board yes) (dnp no)
     (property "Reference" "XL11" (at 205.74 185.42 0)
       (effects (font (size 1.016 1.016)) (justify left))
@@
       (effects (font (size 1.27 1.27)) hide)
     )
+    (property "Price" "40" (at 326.39 48.26 0)
+      (effects (font (size 1.27 1.27)) hide)
+    )
     (pin "1")
     (pin "2")
@@
   )
   (symbol (lib_id "Connectors_kl:SOCKET_2") (at 372.11 35.56 0) (mirror y) (unit 1)
-    (in_bom yes) (on_board yes) (dnp no)
+    (in_bom no) (on_board yes) (dnp no)
     (property "Reference" "XL2" (at 373.38 31.75 0)
       (effects (font (size 1.016 1.016)) (justify left))
@@
   )
   (symbol (lib_id "Connectors_kl:SOCKET_3") (at 219.71 273.05 0) (mirror y) (unit 1)
-    (in_bom yes) (on_board yes) (dnp no)
+    (in_bom no) (on_board yes) (dnp no)
     (property "Reference" "XL20" (at 220.98 278.13 0)
       (effects (font (size 1.016 1.016)) (justify left))
@@
   )
   (symbol (lib_id "Connectors_kl:SOCKET_3") (at 331.47 198.12 0) (unit 1)
-    (in_bom yes) (on_board yes) (dnp no) (fields_autoplaced)
+    (in_bom no) (on_board yes) (dnp no) (fields_autoplaced)
     (property "Reference" "XL13" (at 336.55 196.85 0)
       (effects (font (size 1.016 1.016)) (justify left))
@@
   )
   (symbol (lib_id "Connectors_kl:SOCKET_4") (at 85.09 39.37 0) (mirror y) (unit 1)
-    (in_bom yes) (on_board yes) (dnp no)
+    (in_bom no) (on_board yes) (dnp no)
     (property "Reference" "XL3" (at 85.09 33.02 0)
       (effects (font (size 1.016 1.016)))
@@
       (effects (font (size 1.27 1.27)) hide)
     )
+    (property "Price" "40" (at 344.17 55.88 0)
+      (effects (font (size 1.27 1.27)) hide)
+    )
     (pin "1")
     (pin "2")
@@
   )
   (symbol (lib_id "Tittar_kl:R") (at 302.26 53.34 90) (unit 1)
-    (in_bom yes) (on_board yes) (dnp no)
+    (in_bom no) (on_board yes) (dnp no)
     (property "Reference" "R3" (at 302.26 55.88 90)
       (effects (font (size 1.27 1.27)))
@@
   )
   (symbol (lib_id "Connectors_kl:SOCKET_3") (at 207.01 208.28 0) (unit 1)
-    (in_bom yes) (on_board yes) (dnp no)
+    (in_bom no) (on_board yes) (dnp no)
     (property "Reference" "XL15" (at 205.74 213.36 0)
       (effects (font (size 1.016 1.016)) (justify left))
@@
   )
   (symbol (lib_id "Connectors_kl:SOCKET_2") (at 354.33 91.44 0) (unit 1)
-    (in_bom yes) (on_board yes) (dnp no)
+    (in_bom no) (on_board yes) (dnp no)
     (property "Reference" "XL6" (at 354.33 95.25 0)
       (effects (font (size 1.016 1.016)) (justify left))
@@
   )
   (symbol (lib_id "Connectors_kl:SOCKET_2") (at 354.33 35.56 0) (unit 1)
-    (in_bom yes) (on_board yes) (dnp no)
+    (in_bom no) (on_board yes) (dnp no)
     (property "Reference" "XL1" (at 353.06 31.75 0)
       (effects (font (size 1.016 1.016)) (justify left))
@@
   )
   (symbol (lib_name "REFPOINT_1") (lib_id "pcb_details:REFPOINT") (at 302.26 229.87 0) (unit 1)
-    (in_bom yes) (on_board yes) (dnp no)
+    (in_bom no) (on_board yes) (dnp no)
     (property "Reference" "RP4" (at 306.07 228.6 0)
       (effects (font (size 1.524 1.524)) (justify left))
@@
   )
   (symbol (lib_id "Connectors_kl:SOCKET_4") (at 85.09 64.77 0) (mirror y) (unit 1)
-    (in_bom yes) (on_board yes) (dnp no)
+    (in_bom no) (on_board yes) (dnp no)
     (property "Reference" "XL5" (at 85.09 58.42 0)
       (effects (font (size 1.016 1.016)))
@@
   )
   (symbol (lib_id "Transistors_kl:NPN") (at 287.02 102.87 0) (unit 1)
-    (in_bom yes) (on_board yes) (dnp no) (fields_autoplaced)
+    (in_bom no) (on_board yes) (dnp no) (fields_autoplaced)
     (property "Reference" "Q3" (at 290.83 102.235 0)
       (effects (font (size 1.27 1.27)) (justify left))
@@
   )
   (symbol (lib_id "Connectors_kl:SOCKET_2") (at 372.11 91.44 0) (mirror y) (unit 1)
-    (in_bom yes) (on_board yes) (dnp no)
+    (in_bom no) (on_board yes) (dnp no)
     (property "Reference" "XL7" (at 372.11 95.25 0)
       (effects (font (size 1.016 1.016)) (justify left))
@@
   )
   (symbol (lib_id "Connectors_kl:SOCKET_3") (at 356.87 198.12 0) (mirror y) (unit 1)
-    (in_bom yes) (on_board yes) (dnp no) (fields_autoplaced)
+    (in_bom no) (on_board yes) (dnp no) (fields_autoplaced)
     (property "Reference" "XL14" (at 351.79 196.85 0)
       (effects (font (size 1.016 1.016)) (justify left))

Commit message: Layout started
Parts:
- removed DD1: STM32F072RxTx, LQFP_TQFP:LQFP64, symbol st_kl:STM32F072RxTx
- removed Q1, Q2: NSS20101, SOT:SC89-3, symbol Transistors_kl:NPN
- removed XL3: SOCKET_4, Connectors:PLS-4, symbol Connectors_kl:SOCKET_4
- added C22, C5, C7: 0.1u, Capacitors:CAP_0402_Fab, symbol Tittar_kl:C
- added C23: 10u, Capacitors:CAP_0603_Silks, symbol Tittar_kl:C
- added C3: 2u2, Capacitors:CAP_0603_Silks, symbol Tittar_kl:C
- added DA1: 74VHC1GT125, SOT:SOT23-5, symbol standard_logic:1xBUF_W3STATE
- added DD1: GD32E103CB, LQFP_TQFP:LQFP48, symbol GD:GD32E103CB
- added DD2: W25Q32JV, SO_DIL_TSSOP:SO8_208MIL, symbol Memory:W25Q32JV
- added DD3: MAX98357A, QFN_DFN:QFN-16_EP_3x3_Pitch0.5mm, symbol Audio_kl:MAX98357
- added HOLE2, HOLE4, HOLE6, HOLE8: HOLE_METALLED, PCB:Hole2d7_out4d2mm, symbol pcb_details:HOLE_METALLED
- added R2: 5k1, Resistors:RES_0402_Fab, symbol Tittar_kl:R
- added R5: 1k, Resistors:RES_0402_Fab, symbol Tittar_kl:R
- added R7: 2R0, Resistors:RES_0402_Fab, symbol Tittar_kl:R
- added TP1, TP2, TP3, TP4, TP5: TESTPOINT, PCB:TESTPOINT_1MM, symbol pcb_details:TESTPOINT
- added XL12, XL13: SOCKET_1, Connectors:PLS-1Oval, symbol Connectors_kl:SOCKET_1
- added XL4: USB_C, Connectors:USBC_24PF-009, symbol Connectors_kl:USB_C
- added XL6: SOCKET_4, Connectors:PLS-4-NoHole, symbol Connectors_kl:SOCKET_4
- added XL9: SOCKET_3, Connectors:PLS-3-PAD, symbol Connectors_kl:SOCKET_3
- C10: renamed from C5; value 10u -> 6v3
- C11: renamed from C7; footprint Capacitors:CAP_0603_Silks -> Capacitors:CAP_0402_Fab
- C12: renamed from C8; footprint Capacitors:CAP_0603_Silks -> Capacitors:CAP_0402_Fab
- C13: renamed from C9; footprint Capacitors:CAP_0603_Silks -> Capacitors:CAP_0402_Fab
- C14: renamed from C10; footprint Capacitors:CAP_0603_Silks -> Capacitors:CAP_0402_Fab
- C15: renamed from C4; footprint Capacitors:CAP_0603_Silks -> Capacitors:CAP_0402_Fab
- C16: renamed from C15; footprint Capacitors:CAP_0603_Silks -> Capacitors:CAP_0402_Fab
- C18: renamed from C14; footprint Capacitors:CAP_0603_Silks -> Capacitors:CAP_0402_Fab
- C2, C20: footprint Capacitors:CAP_0603_Silks -> Capacitors:CAP_0402_Fab
- C24: renamed from C16; footprint Capacitors:CAP_0603_Silks -> Capacitors:CAP_0402_Fab
- C4: renamed from C3; footprint Capacitors:CAP_0603_Silks -> Capacitors:CAP_0402_Fab
- C6: value 0.1u -> 1u; footprint Capacitors:CAP_0603_Silks -> Capacitors:CAP_0402_Fab
- C8: renamed from C12; footprint Capacitors:CAP_0603_Silks -> Capacitors:CAP_0402_Fab
- C9: renamed from C11; footprint Capacitors:CAP_0603_Silks -> Capacitors:CAP_0402_Fab
- HOLE1: footprint PCB:Oval7d7x5d7wHole5d5x3d5 -> PCB:Hole2d7_out4d2mm
- HOLE10: renamed from HOLE6; footprint PCB:Oval7d7x5d7wHole5d5x3d5 -> PCB:Hole2d7_out4d2mm
- HOLE11: renamed from HOLE7; footprint PCB:Oval7d7x5d7wHole5d5x3d5 -> PCB:Hole2d7_out4d2mm
- HOLE12: renamed from HOLE8; footprint PCB:Oval7d7x5d7wHole5d5x3d5 -> PCB:Hole2d7_out4d2mm
- HOLE13: renamed from HOLE9; footprint PCB:Oval7d7x5d7wHole5d5x3d5 -> PCB:Hole4_out5d3mm
- HOLE14: renamed from HOLE10; footprint PCB:Oval7d7x5d7wHole5d5x3d5 -> PCB:Hole4_out5d3mm
- HOLE15: renamed from HOLE11; footprint PCB:Oval7d7x5d7wHole5d5x3d5 -> PCB:Hole4_out5d3mm
- HOLE16: renamed from HOLE12; footprint PCB:Oval7d7x5d7wHole5d5x3d5 -> PCB:Hole4_out5d3mm
- HOLE3: renamed from HOLE2; footprint PCB:Oval7d7x5d7wHole5d5x3d5 -> PCB:Hole2d7_out4d2mm
- HOLE5: renamed from HOLE3; footprint PCB:Oval7d7x5d7wHole5d5x3d5 -> PCB:Hole2d7_out4d2mm
- HOLE7: renamed from HOLE4; footprint PCB:Oval7d7x5d7wHole5d5x3d5 -> PCB:Hole2d7_out4d2mm
- HOLE9: renamed from HOLE5; footprint PCB:Oval7d7x5d7wHole5d5x3d5 -> PCB:Hole2d7_out4d2mm
- R1: renamed from R2; footprint Resistors:RES_0603 -> Resistors:RES_0402_Fab
- R10: renamed from R5; footprint Resistors:RES_0603 -> Resistors:RES_0402_Fab
- R11: renamed from R8; footprint Resistors:RES_0603 -> Resistors:RES_0402_Fab
- R12: renamed from R9; footprint Resistors:RES_0603 -> Resistors:RES_0402_Fab
- R13: renamed from R10; footprint Resistors:RES_0603 -> Resistors:RES_0402_Fab
- R14: renamed from R11; footprint Resistors:RES_0603 -> Resistors:RES_0402_Fab
- R15: renamed from R12; footprint Resistors:RES_0603 -> Resistors:RES_0402_Fab
- R16: renamed from R13; footprint Resistors:RES_0603 -> Resistors:RES_0402_Fab
- R17: renamed from R14; footprint Resistors:RES_0603 -> Resistors:RES_0402_Fab
- R18: renamed from R15; footprint Resistors:RES_0603 -> Resistors:RES_0402_Fab
- R19: renamed from R16; footprint Resistors:RES_0603 -> Resistors:RES_0402_Fab
- R20: renamed from R17; footprint Resistors:RES_0603 -> Resistors:RES_0402_Fab
- R21: renamed from R18; footprint Resistors:RES_0603 -> Resistors:RES_0402_Fab
- R22: renamed from R19; footprint Resistors:RES_0603 -> Resistors:RES_0402_Fab
- R23: renamed from R20; footprint Resistors:RES_0603 -> Resistors:RES_0402_Fab
- R24: renamed from R21; footprint Resistors:RES_0603 -> Resistors:RES_0402_Fab
- R25: renamed from R22; footprint Resistors:RES_0603 -> Resistors:RES_0402_Fab
- R26: renamed from R23; footprint Resistors:RES_0603 -> Resistors:RES_0402_Fab
- R27: renamed from R24; footprint Resistors:RES_0603 -> Resistors:RES_0402_Fab
- R3: value DNM -> 5k1; footprint Resistors:RES_0603 -> Resistors:RES_0402_Fab; now in the parts list
- R4: footprint Resistors:RES_0603 -> Resistors:RES_0402_Fab
- R6: renamed from R1; footprint Resistors:RES_0603 -> Resistors:RES_0402_Fab
- R8: renamed from R6; footprint Resistors:RES_0603 -> Resistors:RES_0402_Fab
- R9: renamed from R7; footprint Resistors:RES_0603 -> Resistors:RES_0402_Fab
- XL5: footprint Connectors:PLS-4 -> Connectors:PLS-4-NoHole; now in the parts list
- renumbered C19 to C17, C13 to C19, C17 to C25, C18 to C26, D2 to D1, D1 to D2, DA1 to DA2, Q3 to Q1, Q9 to Q10, Q13 to Q11, Q4 to Q2, Q5 to Q3, Q6 to Q4, Q7 to Q5, Q8 to Q6, Q10 to Q7, Q11 to Q8, Q12 to Q9, RP3 to RP2, RP2 to RP3, XL4 to XL1, XL8 to XL10, XL9 to XL11, XL11 to XL14, XL12 to XL15, XL13 to XL16, XL14 to XL17, XL15 to XL18, XL16 to XL19, XL1 to XL2, XL10 to XL20, XL17 to XL21, XL18 to XL22, XL19 to XL23, XL20 to XL24, XL2 to XL3, XL6 to XL7, XL7 to XL8
Connections:
- net +PwrMCU: now also C7.1, DD1.1 (VBAT), DD1.24 (VDD1), DD1.36 (VDD2), DD1.48 (VDD3), DD1.9 (VDDA), DD2.8 (VCC)
- net Buzzer: now also DD1.27 (PB14)
- net GND: now also R3.2, C22.2, C23.1, C3.2, C5.2, C7.2, DA1.1 (~{OE}), DA1.3 (GND), DD1.23 (VSS1), DD1.35 (VSS2), DD1.44 (BOOT0), DD1.47 (VSS3), DD1.8 (VSSA), DD2.4 (GND), DD3.11 (GND), DD3.15 (GND), DD3.2 (GAIN_SLOT), DD3.3 (GND), DD3.PAD (GND), HOLE2.H, HOLE4.H, HOLE6.H, HOLE8.H, R2.1, XL4.A1 (GND), XL4.A12 (GND), XL4.B1 (GND), XL4.B12 (GND), XL6.1, XL9.1
- net IR_LED_DAC: now also DD1.14 (PA4)
- net IR_LED_IN: no longer R3.2
- net IR_RCVR: now also DD1.11 (PA1)
- net Input1: now also XL5.2, DD1.20 (PB2)
- net Input2: now also XL5.3, DD1.21 (PB10)
- net Input3: now also XL5.4, DD1.22 (PB11)
- net LED_FRONT1: now also DD1.45 (PB8)
- net LED_FRONT2: now also DD1.46 (PB9)
- net LED_PWM1_IN: now also DD1.16 (PA6)
- net LED_PWM2_IN: now also DD1.17 (PA7)
- net LED_PWM3_IN: now also DD1.18 (PB0)
- net LED_PWM4_IN: now also DD1.19 (PB1)
- net Output1: now also DD1.15 (PA5), XL6.2; no longer XL5.2
- net Output2: now also DD1.29 (PA8), XL6.3; no longer XL5.3
- net Output3: now also DD1.3 (PC14), XL6.4; no longer XL5.4
- net SWCLK: now also DD1.37 (SWCLK)
- net SWDIO: now also DD1.34 (SWDIO)
- net UART_RX: now also DD1.13 (PA3)
- net UART_TX: now also DD1.12 (PA2)
- net at R10.2: now also DD1.6 (OSCOUT)
- net at C4.1, XTAL1.1: now also DD1.5 (OSCIN)
- net at R6.2: now also DD1.31 (PA10)
- net IR_LED_TIM renamed USB_CC2
- net USB_CC2: now also XL4.B5 (CC2)
- new net: DD1.30 (PA9), R5.2
- new net: C3.1, R7.2
- new net +5vUSB: R5.1, R7.1, XL4.A4 (VBUS), XL4.A9 (VBUS), XL4.B4 (VBUS), XL4.B9 (VBUS)
- new net +AU_PWR: C22.1, C23.2, DD3.7 (VDD), DD3.8 (VDD)
- new net +NPX_PWR: C5.1, DA1.5 (Vcc), XL9.3
- new net AU_BCLK: DD1.26 (PB13), DD3.16 (BCLK), TP2.1
- new net AU_LRCK: DD1.25 (PB12), DD3.14 (LRCK), TP4.1
- new net AU_SDIN: DD1.28 (PB15), DD3.1 (DIN), TP3.1
- new net AU_SDMODE: DD1.2 (PC13), DD3.4 (~{SD_MODE}), TP5.1
- new net FLASH_IO2: DD1.42 (PB6), DD2.3 (IO2)
- new net FLASH_IO3: DD1.43 (PB7), DD2.7 (IO3)
- new net FLASH_MISO: DD1.40 (NJTRST), DD2.2 (DO/IO1)
- new net FLASH_MOSI: DD1.41 (PB5), DD2.5 (DI/IO0)
- new net FLASH_NSS: DD1.38 (JTDI), DD2.1 (~{CS})
- new net FLASH_SCK: DD1.39 (JTDO), DD2.6 (CLK)
- new net NPX_CTRL: DA1.2 (InA), DD1.10 (PA0), TP1.1
- new net NPX_DATA: DA1.4 (OutY), XL9.2
- new net SPK_M: DD3.10 (OUTN), XL13.1
- new net SPK_P: DD3.9 (OUTP), XL12.1
- new net USB_CC1: R2.2, XL4.A5 (CC1)
- new net USB_D+: DD1.33 (PA12), XL4.A6 (D+), XL4.B6 (D+)
- new net USB_D-: DD1.32 (PA11), XL4.A7 (D-), XL4.B7 (D-)
- no-connect marks 29 -> 16
Other:
- note added: "Audio"
- note added: "Flash Memory"
- note added: "Gain=12, Slot=0"
- note added: "IR TX: DAC0 & TIM6 UART: USART1 SPI0: FLASH SPI1: I2S IR RX: T1C1 SysLED: T0 C2 SideLEDs: T2 C0,1,2,3 FrontLEDs: T3 C2,3 WS2812: T4 C0 Buzzer: T11 C0 DMA0: C1 - SPI0 RX C2 - SPI0 TX C4 - I2S1 TX C5 - U1 RX C6 - U1 TX DMA1: C1 - T4UP C2 - DAC0 C4 - T4C0"
- note added: "NPX Buffer"
- note added: "Outputs Open-Drain"
- note added: "TODO: 1) Who powers NPX? 2) Who powewrs sound?"
- note added: "USB connector"
- note removed: "5VTol"
- note removed: "Alternate SOT23 Footprint"
- note removed: "Outputs Open-Drain 5V Tolerant"
- note removed: "Periphery TIM1 Ch1 - Buzzer TIM2 Ch1 - SysLED Ch2 - LED_Front1 Ch3 - LED_Front2 TIM3 - Indication LEDs TIM6, TIM7 - IR TX TIM14 - System Timer TIM15 - IR RX TIM16, TIM17 - spare IR TX"
- moved on the sheet: BZ1, C1, C10, C11, C12, C13, C14, C15, C2, C24, C25, C26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
