File: IR_PCB_hw/IR_PCB.kicad_sch (KiCad schematic)
At the start: 133 parts, among them Q1 M28S, Q10 SI2303, Q11 SI2303, Q2 M28S, Q3 TSOP48xx, Q4 TSOP48xx, Q5 SI2303, Q6 TSOP48xx, Q7 SI2303, Q8 SI2303, Q9 SI2303

Commit message: Layout in progress
Parts:
- removed C11: 0.1u, Capacitors:CAP_0402_Fab, symbol Tittar_kl:C
- removed TP1: TESTPOINT, PCB:TESTPOINT_1MM, symbol pcb_details:TESTPOINT
- removed XL11, XL7, XL8: SOCKET_2, Connectors:PLS-2, symbol Connectors_kl:SOCKET_2
- removed XL12, XL13: SOCKET_1, Connectors:PLS-1Oval, symbol Connectors_kl:SOCKET_1
- removed XL5, XL6: SOCKET_4, Connectors:PLS-4-NoHole, symbol Connectors_kl:SOCKET_4
- added D13: PMEG2020, Diodes:SOD323, symbol Tittar_kl:D_Shottky
- added R29: 10k, Resistors:RES_0402_Fab, symbol Tittar_kl:R
- added XL5: SOCKET_5, Connectors:SLD_5_2D5_SMD, symbol Connectors_kl:SOCKET_5
- added XL7: SOCKET_3, Connectors:SLD_3_2D5_SMD, symbol Connectors_kl:SOCKET_3
- added XL8: SOCKET_3, Connectors:PLS-3, symbol Connectors_kl:SOCKET_3
- C10: value 6v3 -> 10u; Voltage 10V -> 6v3
- XL1: footprint Connectors:PLS-6_LOCK -> Connectors:PLS-6-NoHole
- XL10, XL2: footprint Connectors:PLS-2 -> Connectors:SLD_2_2D5_SMD
- XL14, XL16, XL18, XL21, XL23: footprint Connectors:PLS-3 -> Connectors:SLD_3_2D5_SMD
- XL9: footprint Connectors:PLS-3-PAD -> Connectors:SLD_3_2D5_SMD
Connections:
- net +BATT is gone; now on net +PwrUnst: C24.1, C25.1, DA2.3 (IN), Q10.2 (S)
- net +NPX_PWR is gone; now on net +PwrUnst: C5.1, DA1.5 (Vcc), XL9.3
- net +5vUSB: now also Q10.1 (G), D13.A, R29.1
- net GND: now also R29.2, XL5.1, XL7.1, XL8.1; no longer Q10.1 (G), XL10.2
- net LED_FRONT1: now also XL7.2, XL8.2
- net LED_FRONT2: now also XL7.3, XL8.3
- net LED_PWM1: now also XL14.3, XL15.3, XL21.3, XL22.3
- net LED_PWM2: now also XL14.2, XL15.2, XL21.2, XL22.2
- net LED_PWM3: now also XL18.3, XL19.3, XL23.3, XL24.3
- net LED_PWM4: now also XL18.2, XL19.2, XL23.2, XL24.2
- net SPK_M: now also XL10.2
- net SPK_P: now also XL10.1
- net at D6.A, R15.2: no longer XL14.2, XL15.2
- net at D5.A, R13.2: no longer XL14.3, XL15.3
- net at D8.A, R20.2: no longer XL18.2, XL19.2
- net at D10.A, R23.2: no longer XL21.2, XL22.2
- net at D9.A, R22.2: no longer XL21.3, XL22.3
- net at D11.A, R26.2: no longer XL23.3, XL24.3
- net at D12.A, R27.2: no longer XL23.2, XL24.2
- net at D4.A, R9.2: no longer XL10.1
- net at D7.A, R17.2: no longer XL18.3, XL19.3
- net +AU_PWR renamed +PwrUnst
- net +PwrUnst: now also D13.C
- net Input1 renamed Gpio1
- net Gpio1: now also XL5.2
- net Input2 renamed Gpio2
- net Gpio2: now also XL5.3
- net Input3 renamed Gpio3
- net Gpio3: now also XL5.4
- net Output1: no longer names the net of DD1.15 (PA5)
- net Output2 renamed Gpio4
- net Gpio4: now also XL5.5
- net Output3: no longer names the net of DD1.3 (PC14)
- no-connect marks 16 -> 18
Other:
- note added: "Battery or USB, and Reverse Current Protection"
- note added: "GPIOs 5V Tolerant"
- note added: "USB detect"
- note removed: "Inputs 5V Tolerant"
- note removed: "Outputs Open-Drain"
- note removed: "Reverse Current Protection"
- moved on the sheet: C1, C10, C2, C24, C25, C26, C8, C9, D1, D10, D11, D12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

Commit message: PCBv3 sent to factory
Parts:
- added Logo1: Logo, Pictures:KiberiadaTYUKF, symbol pcb_details:Logo
- C10, C23, C26: footprint Capacitors:CAP_0603_Silks -> Capacitors:CAP_0603_Fab
- C25: footprint Capacitors:CAP_0805 -> Capacitors:CAP_0603_Fab; Voltage 20V -> 10V
- C3: footprint Capacitors:CAP_0603_Silks -> Capacitors:CAP_0402_Fab
- L1: footprint Inductors:IND_0402 -> Inductors:IND_0402_Fab
Connections:
- net +3v3: no longer XL1.1
- net +PwrMCU: now also XL1.1
Other:
- note removed: "TODO: 1) Who powers NPX? 2) Who powewrs sound?"
- title: IR PCB -> IR PCB v3
Changed lines of the file:
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@@
   (paper "A3")
   (title_block
-    (title "IR PCB")
-    (date "2023-08-05")
+    (title "IR PCB v3")
+    (date "2023-10-07")
     (rev "1")
   )
@@
     (effects (font (size 3 3) (thickness 0.6) bold) (justify left bottom))
   )
-  (text "TODO:\n1) Who powers NPX?\n2) Who powewrs sound?" (at 63.5 25.4 0)
-    (effects (font (size 1.27 1.27)) (justify left bottom))
-  )
   (text "GPIOs\n5V Tolerant" (at 20.32 59.69 0)
     (effects (font (size 1.27 1.27) bold) (justify left bottom))
@@
     )
   )
+  (symbol (lib_id "pcb_details:Logo") (at 316.23 242.57 0) (unit 1)
+    (in_bom no) (on_board yes) (dnp no) (fields_autoplaced)
+    (property "Reference" "Logo1" (at 323.85 241.935 0)
+      (effects (font (size 1.524 1.524)) (justify left))
+    )
+    (property "Value" "Logo" (at 323.85 244.475 0)
+      (effects (font (size 1.524 1.524)) (justify left))
+    )
+    (property "Footprint" "Pictures:KiberiadaTYUKF" (at 316.23 242.57 0)
+      (effects (font (size 1.524 1.524)) hide)
+    )
+    (property "Datasheet" "" (at 316.23 242.57 0)
+      (effects (font (size 1.524 1.524)) hide)
+    )
+    (instances
+      (project "IR_PCB"
+        (path "/26b21aaa-6dc4-45a1-9290-a267c2da2d18"
+          (reference "Logo1") (unit 1)
+        )
+      )
+    )
+  )
   (symbol (lib_id "Tittar_kl:R") (at 227.33 198.12 90) (unit 1)
     (in_bom yes) (on_board yes) (dnp no)
@@
       (effects (font (size 1.27 1.27)) (justify left))
     )
-    (property "Footprint" "Capacitors:CAP_0603_Silks" (at 92.71 180.34 90)
+    (property "Footprint" "Capacitors:CAP_0603_Fab" (at 92.71 180.34 90)
       (effects (font (size 0.7112 0.7112)) (justify bottom) hide)
     )
@@
     )
   )
-  (symbol (lib_id "power:+3v3") (at 26.67 24.13 0) (unit 1)
-    (in_bom yes) (on_board yes) (dnp no)
-    (property "Reference" "#PWR01" (at 26.67 25.146 0)
-      (effects (font (size 0.762 0.762)) hide)
-    )
-    (property "Value" "+3v3" (at 27.94 22.86 0)
-      (effects (font (size 0.762 0.762)))
-    )
-    (property "Footprint" "" (at 26.67 24.13 0)
-      (effects (font (size 1.524 1.524)))
-    )
-    (property "Datasheet" "" (at 26.67 24.13 0)
-      (effects (font (size 1.524 1.524)))
-    )
-    (pin "1")
-    (instances
-      (project "IR_PCB"
-        (path "/26b21aaa-6dc4-45a1-9290-a267c2da2d18"
-          (reference "#PWR01") (unit 1)
-        )
-      )
-    )
-  )
   (symbol (lib_id "Tittar_kl:R") (at 227.33 254 90) (unit 1)
     (in_bom yes) (on_board yes) (dnp no)
@@
       (effects (font (size 1.27 1.27)) (justify left))
     )
-    (property "Footprint" "Capacitors:CAP_0603_Silks" (at 242.57 74.93 90)
+    (property "Footprint" "Capacitors:CAP_0402_Fab" (at 242.57 74.93 90)
       (effects (font (size 0.7112 0.7112)) (justify bottom) hide)
     )
@@
       (effects (font (size 1.016 1.016)))
     )
-    (property "Footprint" "Inductors:IND_0402" (at 87.884 265.684 90)
+    (property "Footprint" "Inductors:IND_0402_Fab" (at 87.884 265.684 90)
       (effects (font (size 1.016 1.016)) hide)
     )
@@
       (effects (font (size 1.27 1.27)) (justify left))
     )
-    (property "Footprint" "Capacitors:CAP_0805" (at 33.02 274.32 90)
+    (property "Footprint" "Capacitors:CAP_0603_Fab" (at 33.02 274.32 90)
       (effects (font (size 0.7112 0.7112)) (justify bottom) hide)
     )
@@
       (effects (font (size 1.27 1.27)) hide)
     )
-    (property "Voltage" "20V" (at 30.48 270.51 0)
+    (property "Voltage" "10V" (at 30.48 270.51 0)
       (effects (font (size 1.27 1.27)) (justify left))
     )
@@
     )
   )
+  (symbol (lib_id "power:+PwrMCU") (at 26.67 24.13 0) (unit 1)
+    (in_bom yes) (on_board yes) (dnp no)
+    (property "Reference" "#PWR01" (at 26.67 22.86 0)
+      (effects (font (size 0.762 0.762)) hide)
+    )
+    (property "Value" "+PwrMCU" (at 27.8384 22.86 0)
+      (effects (font (size 0.762 0.762)))
+    )
+    (property "Footprint" "" (at 26.67 24.13 0)
+      (effects (font (size 1.524 1.524)))
+    )
+    (property "Datasheet" "" (at 26.67 24.13 0)
+      (effects (font (size 1.524 1.524)))
+    )
+    (pin "1")
+    (instances
+      (project "IR_PCB"
+        (path "/26b21aaa-6dc4-45a1-9290-a267c2da2d18"
+          (reference "#PWR01") (unit 1)
+        )
+      )
+      (project "Avada"
+        (path "/5abad6d7-ce46-488e-93d1-8baa746e0378"
+          (reference "#PWR?") (unit 1)
+        )
+      )
+    )
+  )
   (symbol (lib_id "power:GND") (at 292.1 283.21 0) (unit 1)
     (in_bom yes) (on_board yes) (dnp no) (fields_autoplaced)
@@
       (effects (font (size 1.27 1.27)) (justify left))
     )
-    (property "Footprint" "Capacitors:CAP_0603_Silks" (at 63.5 274.32 90)
+    (property "Footprint" "Capacitors:CAP_0603_Fab" (at 63.5 274.32 90)
       (effects (font (size 0.7112 0.7112)) (justify bottom) hide)
     )
@@
       (effects (font (size 1.27 1.27)) (justify left))
     )
-    (property "Footprint" "Capacitors:CAP_0603_Silks" (at 55.88 125.73 90)
+    (property "Footprint" "Capacitors:CAP_0603_Fab" (at 55.88 125.73 90)
       (effects (font (size 0.7112 0.7112)) (justify bottom) hide)
     )

Commit message: PCB v 3.1
Parts:
- C1: value 470uF -> 220uF; PN TAJD477K006RNJ -> 293D227X96R3D2TE3; Price 45 -> 39; Voltage (none) -> 6v3
- C2: Dielectric X5R or X7R -> X7R; PN - -> CC0402KRX7R7BB104; Tolerance 20% -> 10%; Voltage 10V -> 16V
Changed lines of the file:
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@@
       (effects (font (size 1.27 1.27)) (justify left))
     )
-    (property "Value" "470uF" (at 295.91 35.56 0)
+    (property "Value" "220uF" (at 295.91 35.56 0)
       (effects (font (size 1.27 1.27)) (justify left))
     )
@@
       (effects (font (size 1.27 1.27)) hide)
     )
-    (property "PN" "TAJD477K006RNJ" (at 304.8 34.29 0)
+    (property "PN" "293D227X96R3D2TE3" (at 304.8 34.29 0)
       (effects (font (size 1.27 1.27)) hide)
     )
-    (property "Price" "45" (at 304.8 34.29 0)
+    (property "Price" "39" (at 304.8 34.29 0)
+      (effects (font (size 1.27 1.27)) hide)
+    )
+    (property "Voltage" "6v3" (at 304.8 34.29 0)
+      (effects (font (size 1.27 1.27)))
+    )
+    (property "Description" "Cap Tant Solid 220uF 6.3V D CASE" (at 304.8 34.29 0)
       (effects (font (size 1.27 1.27)) hide)
     )
@@
       (effects (font (size 1.27 1.27)) hide)
     )
-    (property "PN" "-" (at 317.5 34.29 0)
+    (property "PN" "CC0402KRX7R7BB104" (at 317.5 34.29 0)
       (effects (font (size 1.27 1.27)) hide)
     )
@@
       (effects (font (size 1.27 1.27)) hide)
     )
-    (property "Dielectric" "X5R or X7R" (at 317.5 34.29 0)
+    (property "Dielectric" "X7R" (at 317.5 34.29 0)
       (effects (font (size 1.27 1.27)) hide)
     )
-    (property "Tolerance" "20%" (at 317.5 34.29 0)
+    (property "Tolerance" "10%" (at 317.5 34.29 0)
       (effects (font (size 1.27 1.27)) hide)
     )
-    (property "Voltage" "10V" (at 317.5 34.29 0)
+    (property "Voltage" "16V" (at 317.5 34.29 0)
       (effects (font (size 1.27 1.27)) (justify left))
     )

Commit message: working on bom
Parts:
- DD2: value W25Q32JV -> W25Q32JVSIQ; Price (none) -> 49; URL (none) -> https://www.chipdip.ru/product/w25q32jvssiq
- Q10, Q11, Q5, Q7, Q8, Q9: value SI2303 -> SI2301
- Q4: value TSOP48xx -> TSOP4856
- XL4: value USB_C -> USB_C 24PF-009; Price (none) -> 40; URL (none) -> https://www.zip-2002.ru/product/usb3-1_type-c_24pf-009/
Changed lines of the file:
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@@
       (effects (font (size 1.27 1.27)))
     )
-    (property "Value" "SI2303" (at 78.74 229.87 0)
+    (property "Value" "SI2301" (at 78.74 229.87 0)
       (effects (font (size 1.27 1.27)))
     )
@@
       (effects (font (size 1.27 1.27)))
     )
-    (property "Value" "USB_C" (at 228.6 27.94 0)
+    (property "Value" "USB_C 24PF-009" (at 228.6 27.94 0)
       (effects (font (size 1.27 1.27)))
     )
@@
       (effects (font (size 1.27 1.27)) hide)
     )
+    (property "URL" "https://www.zip-2002.ru/product/usb3-1_type-c_24pf-009/" (at 228.6 49.53 0)
+      (effects (font (size 1.27 1.27)) hide)
+    )
+    (property "Price" "40" (at 228.6 49.53 0)
+      (effects (font (size 1.27 1.27)) hide)
+    )
     (pin "B1")
     (pin "B10")
@@
       (effects (font (size 1.524 1.524)))
     )
-    (property "Value" "TSOP48xx" (at 314.3333 147.32 0)
+    (property "Value" "TSOP4856" (at 314.3333 147.32 0)
       (effects (font (size 1.524 1.524)))
     )
@@
       (effects (font (size 1.27 1.27)))
     )
-    (property "Value" "SI2303" (at 135.89 184.5564 0)
+    (property "Value" "SI2301" (at 135.89 184.5564 0)
       (effects (font (size 1.27 1.27)))
     )
@@
       (effects (font (size 1.27 1.27)))
     )
-    (property "Value" "SI2303" (at 137.16 237.8964 0)
+    (property "Value" "SI2301" (at 137.16 237.8964 0)
       (effects (font (size 1.27 1.27)))
     )
@@
       (effects (font (size 1.27 1.27)))
     )
-    (property "Value" "SI2303" (at 135.89 157.8864 0)
+    (property "Value" "SI2301" (at 135.89 157.8864 0)
       (effects (font (size 1.27 1.27)))
     )
@@
       (effects (font (size 1.524 1.524)))
     )
-    (property "Value" "W25Q32JV" (at 229.235 107.95 0)
+    (property "Value" "W25Q32JVSIQ" (at 229.235 107.95 0)
       (effects (font (size 1.524 1.524)))
     )
@@
       (effects (font (size 1.524 1.524)) hide)
     )
+    (property "URL" "https://www.chipdip.ru/product/w25q32jvssiq" (at 229.87 118.11 0)
+      (effects (font (size 1.27 1.27)) hide)
+    )
+    (property "Price" "49" (at 229.87 118.11 0)
+      (effects (font (size 1.27 1.27)) hide)
+    )
     (pin "1")
     (pin "2")
@@
       (effects (font (size 1.27 1.27)))
     )
-    (property "Value" "SI2303" (at 137.16 211.2264 0)
+    (property "Value" "SI2301" (at 137.16 211.2264 0)
       (effects (font (size 1.27 1.27)))
     )
@@
       (effects (font (size 1.27 1.27)))
     )
-    (property "Value" "SI2303" (at 375.92 223.9264 0)
+    (property "Value" "SI2301" (at 375.92 223.9264 0)
       (effects (font (size 1.27 1.27)))
     )

Commit message: BOM constructed
Parts:
- removed C15: 18pF, Capacitors:CAP_0402_Fab, symbol Tittar_kl:C
- added C11: 18pF, Capacitors:CAP_0402_Fab, symbol Tittar_kl:C
- BZ1: value PS-9627 -> 9650-5.5R/16R; Price 25 -> 11; URL http://www.quartz1.com/price/model.php?akt=7940.06 -> https://aliexpress.ru/item/1005005350539003.html?spm=a2g2w.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
- C1: value 220uF -> 330uF; PN 293D227X96R3D2TE3 -> (none); Price 39 -> 15; URL (none) -> https://aliexpress.ru/item/32969159998.html?sku_id=66590165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
- C10: Manufacturer - -> Samsung; PN - -> CL10A106MP8NNNC; Price 0.5 -> 1.52; URL (none) -> https://www.promelec.ru/product/335887/; Voltage 6v3 -> 10v
- C17: Dielectric X5R or X7R -> X5R; Manufacturer - -> Samsung; PN GRM31CR60J476ME19L -> CL31A476MQHNNNE; Price 25 -> 5.04; URL https://www.chipdip.ru/product/grm31cr60j476me19l -> https://www.promelec.ru/product/336530/
- C19, C21: Dielectric X5R or X7R -> X5R; Manufacturer - -> Samsung; PN GRM31CR60J476ME19L -> CL31A476MQHNNNE; Price 25 -> 2.36; URL https://www.chipdip.ru/product/grm31cr60j476me19l -> https://www.promelec.ru/product/336530/
- C2: Manufacturer - -> Yageo; Price 0.5 -> 0.17; URL (none) -> https://www.promelec.ru/product/141827/
- C23: Dielectric (none) -> X5R or X7R; Manufacturer (none) -> Samsung; PN CL10A106MQ8NNNC -> CL10A106MP8NNNC; Price 2.5 -> 0.41; Tolerance (none) -> 20%; Type (none) -> Capacitor SMD; URL https://www.terraelectronica.ru/catalog.php?ID=1155&search=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 -> https://www.promelec.ru/product/335887/; Voltage (none) -> 10v
- C25: Manufacturer - -> Samsung; PN - -> CL10A106MP8NNNC; Price 2 -> 0.41; URL (none) -> https://www.promelec.ru/product/335887/; Voltage 10V -> 10v
- C26: Manufacturer - -> Samsung; PN - -> CL10A106MP8NNNC; Price 0.5 -> 0.41; URL (none) -> https://www.promelec.ru/product/335887/; Voltage 10V -> 10v
- C3: Dielectric X5R or X7R -> X5R; Manufacturer - -> Murata; PN - -> GRM155R61A225KE95D; Price 0.5 -> 1.51; Tolerance 20% -> 10%; URL (none) -> https://www.promelec.ru/product/315859/
- C4: Manufacturer - -> Yageo; PN - -> CC0402JRNPO9BN180; Price 0.5 -> 0.48; Tolerance 20% -> 5%; URL (none) -> https://www.promelec.ru/product/188454/; Voltage 10V -> 50V
- C6: Dielectric X5R or X7R -> X5R; Manufacturer - -> Hottech; PN - -> C1005A105K100NT; Price 0.5 -> 0.23; Tolerance 20% -> 10%; URL (none) -> https://www.promelec.ru/product/522035/
- C8: Dielectric X5R or X7R -> X5R; Manufacturer - -> Hottech; PN - -> C1005A105K100NT; Price 0.5 -> 0.13; Tolerance 20% -> 10%; URL (none) -> https://www.promelec.ru/product/522035/
- D1: Price 4 -> 12.59; URL (none) -> https://onelec.ru/products/tsal6200-1a020efd-62ab-4a3f-93a5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
- D10, D11, D12, D5, D6, D7, D8, D9: value BL-L502URC -> ~; Price 4 -> 4.5; URL (none) -> https://aliexpress.ru/item/1005003323749658.html?sku_id=120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
- D13: PN (none) -> PMEG2020AEA,115; Price 5 -> 10.59; URL (none) -> https://onelec.ru/products/pmeg2020aea-115-cdb00143-854a-48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
- D2: value L-C191LBCT -> LTST-C191KGKT; PN L-C191LBCT -> LTST-C191KGKT; Price 4 -> 3.46; URL http://onelec.ru/products/l-c191lbct -> https://www.promelec.ru/product/343092/
- D3, D4: value BL-L522PGC -> ~; Price 4 -> 4.5; URL (none) -> https://aliexpress.ru/item/1005003323749658.html?sku_id=120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
- DA1: Price 5.5 -> 16.15; URL https://www.terraelectronica.ru/catalog.php?ID=301&search=m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 -> https://onelec.ru/products/m74vhc1gt125dt1g-fbb783f3-f3a3-4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
- DA2: Price 19 -> 15.89; URL https://www.chipdip.ru/product/lm1117gs-3.3 -> https://www.promelec.ru/product/479044/
- DD1: Price (none) -> 109.59; URL (none) -> https://www.promelec.ru/product/426829/
- DD2: PN (none) -> W25Q32JVSSIQ; Price 49 -> 26.65; URL https://www.chipdip.ru/product/w25q32jvssiq -> https://www.promelec.ru/product/507481/
- DD3: Price (none) -> 42.63; URL (none) -> https://aliexpress.ru/item/1005005819681447.html?spm=a2g2w.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
- L1: PN - -> BLM15AG102SN1D; Price 4 -> 0.85; URL (none) -> https://www.promelec.ru/product/184235/
- Q1: Price (none) -> 3; now in the parts list
- Q2: now in the parts list
- Q3, Q6: value TSOP48xx -> TSOP4856; Price 120 -> 80.2; URL (none) -> https://onelec.ru/products/tsop4856-c5e4357e-a7a0-42b9-8627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
- Q4: Price 120 -> 80.2; URL (none) -> https://onelec.ru/products/tsop4856-c5e4357e-a7a0-42b9-8627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
- R1: PN - -> RC0402FR-0710KL; Price 0.5 -> 0.2; URL (none) -> https://www.promelec.ru/product/305624/
- R11: PN - -> RC0402FR-0751RL; Price 0.5 -> 0.35; URL (none) -> https://www.promelec.ru/product/305769/
- R2: PN - -> RC0402FR-075K1L; Price 0.5 -> 0.31; URL (none) -> https://www.promelec.ru/product/229745/
- R4: PN - -> RI0402L1001FT; Price 0.5 -> 0.11; URL (none) -> https://www.promelec.ru/product/415937/
- R7: PN - -> RI0402L2R00FT; Price 0.5 -> 0.15; URL (none) -> https://www.promelec.ru/product/529480/
- R8: PN - -> RC0402FR-07100RL; Price 0.5 -> 0.26; URL (none) -> https://www.promelec.ru/product/229700/
- TP2, TP3, TP4, TP5, XL1, XL5, XL7, XL8, XL9: now left out of the parts list
- XTAL1: PN (none) -> SJK-7U-12.000-12-30-80-C-50; Price 15 -> 11.26; URL (none) -> https://www.promelec.ru/product/536327/
Connections:
- net +PwrUnst: now also C23.1; no longer C23.2
- net GND: now also C23.2, C11.2; no longer C23.1
- net at R10.1, XTAL1.2: now also C11.1
